File: high-gain-diff-probe.sch (KiCad schematic (older format))
At the start: 104 parts, among them J1 BANANA, J2 BNC, J3 BANANA, J4 BNC, J5 Conn_Coaxial, J6 Conn_01x03_Female, Q1 BCV49, Q2 BCV48, SW1 ‎MRB24B‎, SW2 ‎MRB24B‎, SW3 SW_SPDT, SW4 SW_DPST_x2, SW5 SW_DP3T, U1 AD8428BRZ, U2 ADA4004, U3 BUF634A, U4 LM393, U5 LM393, U6 LM393

Commit message: Add notes to schematic
Parts:
- added D13, D14: 1N4001, Diode_THT:D_DO-41_SOD81_P10.16mm_Horizontal, symbol Diode:1N4001
- added JP1: BANDWIDTH, symbol Jumper:SolderJumper_2_Open
- J6: value Conn_01x03_Female -> POWER
- RV1: Name (none) -> CM Trim
- SW1: value ‎MRB24B‎ -> MB04L1NCGD; symbol Switch:SW_DP3T -> high-gain-diff-probe:SW_DP4T
- SW2: value ‎MRB24B‎ -> MB04L1NCGD
- SW4: renamed from SW5; value SW_DP3T -> SW_DPST_x2
- gave numbers to parts that had none: 12
Connections:
- net +15V: now also D13.2 (A)
- net -15V: now also D14.1 (K), JP1.2 (B)
- net ATTEN+: now also SW1.B; no longer SW1.7
- net ATTEN-: now also SW1.A (B); no longer SW1.3
- net GND: now also SW1.4 (9), SW1.9
- net HiZ+: now reaches C6.1, R6.1
- net HiZ+: now also SW1.6; no longer SW1.5
- net AC+: now reaches C4.1
- net AC+: now also SW1.7; no longer SW1.6
- net LoZ+: now reaches R4.1, SW1.8 (3)
- net HiZ-: now reaches C5.1, R5.1, SW1.1 (6)
- net AC-: now reaches C3.1, SW1.2 (7)
- net LoZ-: now reaches R3.1
- net LoZ-: now also SW1.3; no longer SW1.4
- net at D7.2 (A), D8.2 (A): now also SW4.3 (A); no longer SW4.1 (A)
- net at C26.2, Q2.1 (C), R19.2: now also SW4.4 (B); no longer SW4.2 (B)
- net at C29.2, D10.2 (A), R19.1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: now also D14.2 (A)
- net at C28.1, D9.1 (K), R18.2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: now also D13.1 (K)
- net at U3.1 (BW): now also JP1.1 (A)
- no-connect marks 3 -> 2
Other:
- note added: "+-12.8V Offset Range\nwith 15V supply."
- note added: "20:1 Attenuator for HiZ inputs.\nProvides return path for INA input bias currents.\nSets corner for AC high-pass (~2Hz)."
- note added: "33ohm resistors ensure protection diodes\nconduct before INA internal diodes, and\nform an RF low-pass filter with the capacitors.\nCould add a ferrite bead as well but be careful\nabout resonance."
- note added: "9V batteries discharge\nin an hour with the\noutput saturated into\n50 ohms.\n\n\n$0.10 per minute."
- note added: "AC coupling caps could hold\ncharge and damage circuits."
- note added: "Adjustable low-pass filter.\nC18: Just tones down very high frequencies.\nC20: 96.5kHz -3dB"
- note added: "Can parallel the input stage of the INA\nwith the filter pins. Can reduce the amp's\nnoise by half in the flatband with 4 amps\nin parallel. Also increases offset voltage\nand source resistance noise, so it makes\nHiZ inputs noisier."
- note added: "Capacitance multiplier reduces noise.\nAlso regulates higher input voltages to 15V.\nD13,D14 protect B-E junctions if power is turned\noff but probe is connected to signal voltage."
- note added: "Default gain of INA is 2000X.\nCould use an SP3T switch."
- note added: "Diode OR Power inputs\nand battery reverse\ncurrent protection."
- note added: "External power input.\nBe careful about the\nground loop between\nscope and power supply."
- note added: "Gold-plated "dry" switch contacts will hopefully\nnot be damaged by the instantaneous voltage/\ncurrent into the attenuator, and will conduct\nvery low level signals without requiring "wetting"."
- note added: "High-current buffer helps drive up\nto 12.5V into 50 ohms and drain 9V\nbatteries quickly."
- note added: "If the differential input voltage is 0.6V or more the\nprotection diodes start to conduct.\n\nThe output saturates well before that due to the high gain."
- note added: "Input overvoltage indicator LEDs.\nDetects when either protection diode\nbecomes forward biased."
- note added: "Low-leakage diodes protect INA inputs from\ncommon mode voltages beyond the supply rails\nand differential voltages above 1V. Can handle\n500mA until they overheat or about 40V to GND\non the LoZ inputs."
- note added: "Output saturation indicator LED.\nDetects when the INA output voltage\nis close to the maximum value."
- note added: "Solder jumper enables high current/high bandwidth\nmode. We don't need the increased bandwidth, but\nit does improve large signal settling time and harmonic\ndistortion significantly. Also increases noise a bit and\nquiescent current of course."
- note added: "TODO: Accurate detent or switch\nto set Ref exactly to GND?"
- note added: "TODO: Invert output?\nHysteresis?\nSize filter caps."
- note removed: "+-12.8V Offset Range"
- note removed: "If the differential input voltage is 0.6V or more the\nprotection diodes start to conduct.\nThe output saturates well before that due to the high gain."
- moved on the sheet: C1, C2, C21, C22, C23, C24, C27, C3, C30, C31, C4, C5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

Commit message: Add footprints to most parts
Parts:
- BT1, BT2, BT3, BT4: footprint (none) -> Connector_Wire:SolderWire-0.5sqmm_1x02_P4.6mm_D0.9mm_OD2.1mm_Relief
- C1, C10, C11, C12, C13, C14, C15, C16, C17, C18, C19, C2, C20, C21, C22, C27, C30, C31, C32, C33, C34, C35, C36, C37, C5, C6, C9: footprint (none) -> Capacitor_SMD:C_0603_1608Metric_Pad1.05x0.95mm_HandSolder
- C23, C24, C28, C29: footprint (none) -> Capacitor_THT:CP_Radial_D6.3mm_P2.50mm; MPN (none) -> 25ML47MEFC6.3X5
- C25, C26: value 1uF -> 100nF; footprint (none) -> Capacitor_SMD:C_0603_1608Metric_Pad1.05x0.95mm_HandSolder
- C3, C4: value 1.5uF 100V -> 1uF FILM; footprint (none) -> high-gain-diff-probe:C_6054_WIMA; MPN (none) -> SMDTF04100YA00JT00
- C7, C8: value 1-3pF -> 3-10pF; footprint (none) -> Capacitor_SMD:C_Trimmer_Voltronics_JZ; MPN (none) -> SGC3S100NM
- D1, D2, D3: footprint (none) -> Package_TO_SOT_SMD:SOT-23
- D15, D16, D17, D6: footprint (none) -> LED_SMD:LED_0603_1608Metric_Pad1.05x0.95mm_HandSolder
- J1, J3: footprint (none) -> Connector:Banana_Jack_1Pin
- J2, J4: footprint (none) -> Connector_Coaxial:BNC_Amphenol_B6252HB-NPP3G-50_Horizontal
- J5: value Conn_Coaxial -> BNC; footprint (none) -> Connector_Coaxial:BNC_Amphenol_B6252HB-NPP3G-50_Horizontal
- JP1: footprint (none) -> Jumper:SolderJumper-2_P1.3mm_Open_TrianglePad1.0x1.5mm
- R1, R10, R11, R12, R13, R14, R15, R17, R18, R19, R2, R20, R21, R22, R23, R24, R25, R26, R27, R5, R6, R7, R8, R9: footprint (none) -> Resistor_SMD:R_0603_1608Metric_Pad0.98x0.95mm_HandSolder
- R16, R3, R4: footprint (none) -> Resistor_SMD:R_1210_3225Metric_Pad1.30x2.65mm_HandSolder
- RV1: footprint (none) -> Potentiometer_THT:Potentiometer_Bourns_3266W_Vertical
- RV2: footprint (none) -> Potentiometer_THT:Potentiometer_Bourns_3296Y_Vertical
- U1, U4, U5, U6: footprint (none) -> Package_SO:SOIC-8_3.9x4.9mm_P1.27mm
Other:
- note added: "Can choose different AC cap depending\non your low frequency, voltage, leakage,\nmicrophonics, and cost priorities."
- note added: "TODO: Check size of pots you have"

Commit message: Add footprints for everything
Parts:
- removed SW2: MB04L1NCGD, symbol Switch:SW_DP3T
- added SW2: MB04L1NCGD, high-gain-diff-probe:SW_DPNT_CK_M, symbol high-gain-diff-probe:SW_DP4T
- J6: footprint (none) -> Connector_PinHeader_2.54mm:PinHeader_1x03_P2.54mm_Horizontal
- SW1: footprint (none) -> high-gain-diff-probe:SW_DPNT_CK_M; MPN (none) -> MB04L1NCGD
- SW3: value SW_SPDT -> GF-626-0061; footprint (none) -> high-gain-diff-probe:SW_CW_GF-626_DPDT; MPN (none) -> GF-626-0061
- SW4: value SW_DPST_x2 -> GF-626-0061; footprint (none) -> high-gain-diff-probe:SW_CW_GF-626_DPDT; symbol Switch:SW_DPST_x2 -> Switch:SW_DPDT_x2; MPN (none) -> GF-626-0061
- U1: MPN (none) -> AD8428BRZ
Connections:
- net AC+: now also SW1.8 (3); no longer SW1.7
- net AC-: now also SW1.3; no longer SW1.2 (7)
- net FIL+: now also SW2.B
- net FIL-: now also SW2.A (B)
- net GND: now also SW1.1 (6), SW1.6; no longer SW1.4 (9), SW1.9
- net HiZ+: now also SW1.9; no longer SW1.6
- net HiZ-: now also SW1.4 (9); no longer SW1.1 (6)
- net LoZ+: now also SW1.7; no longer SW1.8 (3)
- net LoZ-: now also SW1.2 (7); no longer SW1.3
- net RG_500X: now also SW2.2 (7)
- net RG_50X: now also SW2.3
- net at D7.2 (A), D8.2 (A): now also SW4.5 (B); no longer SW4.3 (A)
- net at D4.1 (K), D5.1 (K): now also SW4.2 (B); no longer SW4.1 (A)
- net at C26.2, Q2.1 (C), R19.2: now also SW4.6 (C); no longer SW4.4 (B)
- net at C25.1, D6.2 (A), Q1.2 (C)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: now also SW4.3 (C); no longer SW4.2 (B)
- net at R10.2: now also SW2.7
- net at R9.2: now also SW2.8 (3)
- no-connect marks 2 -> 6
Other:
- moved on the sheet: C1, C2, C3, C4, C5, C6, J1, J2, J3, J4, R1, R10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
