File: high-gain-diff-probe.sch (KiCad schematic (older format))
At the start: 98 parts, among them J1 30V DC IN, J2 BNC, J4 BNC, J5 BNC, K1 FTR-B3SA012Z, K2 FTR-B3SA012Z, Q1 MMBT3906, SW1 MB04L1NCGD, SW2 MB05L1NCGD, SW3 SPDT, SW4 MB04L1NCGD, SW6 SPDT, U1 AD8428BRZ, U2 OP1177AR, U3 BUF634A, U6 LM393, U7 AD8671, U8 BUF634A

Commit message: More layout
Parts:
- added C24, C25: 47uF, Capacitor_SMD:CP_Elec_6.3x7.7, symbol Device:CP1
- added C26, C28, C29, C32, C33, C35: 1uF, Capacitor_SMD:C_0603_1608Metric_Pad1.05x0.95mm_HandSolder, symbol Device:C_Small
- added JP2: BANDWIDTH, Jumper:SolderJumper-2_P1.3mm_Open_TrianglePad1.0x1.5mm, symbol Jumper:SolderJumper_2_Open
Connections:
- net +15V: now also C24.1, C26.1, C29.1, C33.1
- net -15V: now also C25.2, C28.2, C32.2, C35.2, JP2.2 (B)
- net GND: now also J1.MP (MountPin), C24.2, C25.1, C26.2, C28.1, C29.2, C32.1, C33.2, C35.1
- net at U8.1 (BW): now also JP2.1 (A)
Other:
- note added: "Power must be isolated\nfrom ground."
- note removed: "Input must be isolated\nfrom ground."
- moved on the sheet: C15, C16, C21, C23, C27, C30, C31, C38, D11, D12, D7, F4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

Commit message: Tweaks
Parts:
- removed D18, D19: S1A, Diode_SMD:D_SMA_Handsoldering, symbol Diode:1N4001
- removed D7: US1A, Diode_SMD:D_SMA, symbol Diode:US1A
- added D4, D5, D6: DSS15, Diode_SMD:D_SOD-123F, symbol Device:D_Schottky
- R20: value 1k -> 1k 1/4W; footprint Capacitor_SMD:C_0603_1608Metric_Pad1.05x0.95mm_HandSolder -> Resistor_SMD:R_1206_3216Metric_Pad1.30x1.75mm_HandSolder; MPN (none) -> RNCP1206FTD1K00
- R21: value 250k -> 100k; footprint Capacitor_SMD:C_0603_1608Metric_Pad1.05x0.95mm_HandSolder -> Resistor_SMD:R_0603_1608Metric_Pad0.98x0.95mm_HandSolder
- SW2: Name (none) -> Gain Select
Connections:
- net +15V: now also D4.1 (K)
- net -15V: now also D6.2 (A); no longer SW2.B
- net ATTEN_EN: now also D5.1 (K)
- net GND: now also SW2.6, SW2.7, SW2.8 (3), SW2.B
- net at F4.1: now also D4.2 (A)
- net at K1.8, K2.1: now also D5.2 (A), D6.1 (K)
- no-connect marks 10 -> 7
Other:
- note added: "2 12V relays in series to run off\nthe 30V input through a resistor."
- note removed: "2 12V relays in series to run off\nthe 32V input through a resistor."
- moved on the sheet: Q1, R20, R21, SW2B

Commit message: More layout
Parts:
- removed C38: 1uF, Capacitor_SMD:C_0603_1608Metric_Pad1.05x0.95mm_HandSolder, symbol Device:C_Small
Other:
- note added: "TODO: Connect frame of switches to GND"
- moved on the sheet: C29, C32
Changed lines of the file:
@@
-	1    0    0    -1
-$EndComp
-$Comp
-L Device:C_Small C38
-U 1 1 60DEF055
-P 13400 1100
-F 0 "C38" H 13492 1146 50  0000 L CNN
-F 1 "1uF" H 13492 1055 50  0000 L CNN
-F 2 "Capacitor_SMD:C_0603_1608Metric_Pad1.05x0.95mm_HandSolder" H 13438 950 50  0001 C CNN
-F 3 "~" H 13400 1100 50  0001 C CNN
-F 4 "CL10A105KL8NNNC" H 13400 1100 50  0001 C CNN "MPN"
-	1    13400 1100
 	1    0    0    -1
 $EndComp
@@
 L power:+15V #PWR0104
 U 1 1 61B54C2E
-P 13400 700
-F 0 "#PWR0104" H 13400 550 50  0001 C CNN
-F 1 "+15V" H 13400 850 50  0000 C CNN
-F 2 "" H 13400 700 50  0001 C CNN
-F 3 "" H 13400 700 50  0001 C CNN
-	1    13400 700
+P 13500 900
+F 0 "#PWR0104" H 13500 750 50  0001 C CNN
+F 1 "+15V" H 13500 1050 50  0000 C CNN
+F 2 "" H 13500 900 50  0001 C CNN
+F 3 "" H 13500 900 50  0001 C CNN
+	1    13500 900
 	1    0    0    -1
 $EndComp
@@
 L power:-15V #PWR0105
 U 1 1 61B54C34
-P 13400 1500
-F 0 "#PWR0105" H 13400 1600 50  0001 C CNN
-F 1 "-15V" H 13400 1650 50  0000 C CNN
-F 2 "" H 13400 1500 50  0001 C CNN
-F 3 "" H 13400 1500 50  0001 C CNN
-	1    13400 1500
+P 13500 1500
+F 0 "#PWR0105" H 13500 1600 50  0001 C CNN
+F 1 "-15V" H 13500 1650 50  0000 C CNN
+F 2 "" H 13500 1500 50  0001 C CNN
+F 3 "" H 13500 1500 50  0001 C CNN
+	1    13500 1500
 	-1   0    0    1
 $EndComp
@@
 L Device:C_Small C29
 U 1 1 61B54C42
-P 13800 900
-F 0 "C29" H 13892 946 50  0000 L CNN
-F 1 "1uF" H 13892 855 50  0000 L CNN
-F 2 "Capacitor_SMD:C_0603_1608Metric_Pad1.05x0.95mm_HandSolder" H 13838 750 50  0001 C CNN
-F 3 "~" H 13800 900 50  0001 C CNN
-F 4 "CL10A105KL8NNNC" H 13800 900 50  0001 C CNN "MPN"
-	1    13800 900
+P 13500 1000
+F 0 "C29" H 13592 1046 50  0000 L CNN
+F 1 "1uF" H 13592 955 50  0000 L CNN
+F 2 "Capacitor_SMD:C_0603_1608Metric_Pad1.05x0.95mm_HandSolder" H 13538 850 50  0001 C CNN
+F 3 "~" H 13500 1000 50  0001 C CNN
+F 4 "CL10A105KL8NNNC" H 13500 1000 50  0001 C CNN "MPN"
+	1    13500 1000
 	-1   0    0    -1
 $EndComp
@@
 L Device:C_Small C32
 U 1 1 61B54C49
-P 13800 1300
-F 0 "C32" H 13892 1346 50  0000 L CNN
-F 1 "1uF" H 13892 1255 50  0000 L CNN
-F 2 "Capacitor_SMD:C_0603_1608Metric_Pad1.05x0.95mm_HandSolder" H 13838 1150 50  0001 C CNN
-F 3 "~" H 13800 1300 50  0001 C CNN
-F 4 "CL10A105KL8NNNC" H 13800 1300 50  0001 C CNN "MPN"
-	1    13800 1300
+P 13500 1400
+F 0 "C32" H 13592 1446 50  0000 L CNN
+F 1 "1uF" H 13592 1355 50  0000 L CNN
+F 2 "Capacitor_SMD:C_0603_1608Metric_Pad1.05x0.95mm_HandSolder" H 13538 1250 50  0001 C CNN
+F 3 "~" H 13500 1400 50  0001 C CNN
+F 4 "CL10A105KL8NNNC" H 13500 1400 50  0001 C CNN "MPN"
+	1    13500 1400
 	-1   0    0    -1
 $EndComp
-Wire Wire Line
-	13400 1500 13400 1450
-Wire Wire Line
-	13400 1450 13800 1450
-Wire Wire Line
-	13800 1450 13800 1400
-Wire Wire Line
-	13800 800  13800 750
-Wire Wire Line
-	13800 750  13400 750
-Wire Wire Line
-	13400 700  13400 750
-Wire Wire Line
-	13400 750  13400 1000
-Connection ~ 13400 750
-Wire Wire Line
-	13400 1200 13400 1450
-Connection ~ 13400 1450
 $Comp
 L power:GND #PWR0113
 U 1 1 61B54C59
-P 14000 1200
-F 0 "#PWR0113" H 14000 950 50  0001 C CNN
-F 1 "GND" H 14000 1050 50  0000 C CNN
-F 2 "" H 14000 1200 50  0001 C CNN
-F 3 "" H 14000 1200 50  0001 C CNN
-	1    14000 1200
-	1    0    0    -1
-$EndComp
-Wire Wire Line
-	13800 1000 13800 1100
-Wire Wire Line
-	13800 1100 14000 1100
-Wire Wire Line
-	14000 1100 14000 1200
-Connection ~ 13800 1100
-Wire Wire Line
-	13800 1100 13800 1200
+P 13700 1300
+F 0 "#PWR0113" H 13700 1050 50  0001 C CNN
+F 1 "GND" H 13700 1150 50  0000 C CNN
+F 2 "" H 13700 1300 50  0001 C CNN
+F 3 "" H 13700 1300 50  0001 C CNN
+	1    13700 1300
+	1    0    0    -1
+$EndComp
+Wire Wire Line
+	13500 1100 13500 1200
+Wire Wire Line
+	13500 1200 13700 1200
+Wire Wire Line
+	13700 1200 13700 1300
+Connection ~ 13500 1200
+Wire Wire Line
+	13500 1200 13500 1300
 $Comp
 L power:+15V #PWR0114
@@
 Wire Wire Line
 	4600 900  4800 900
+Text Notes 12050 3600 0    50   ~ 0
+TODO: Connect frame of switches to GND
 $EndSCHEMATC

Commit message: Finish Layout
Parts:
- C3, C4: value 2.2uF 63V FILM -> 1uF 100V FILM; footprint Capacitor_THT:C_Rect_L13.5mm_W5.0mm_P10.00mm_FKS3_FKP3_MKS4 -> Capacitor_THT:C_Rect_L7.2mm_W7.2mm_P5.00mm_FKS2_FKP2_MKS2_MKP2; MPN R60DF4220506AJ -> R82EC4100SH70J
- RV2, RV5: MPN PTV09A-4015U-B503 -> PTV09A-4025F-B503
- SW3: symbol Switch:SW_SPDT -> Switch:SW_DPDT_x2
Other:
- moved on the sheet: C18, C20, SW3A
Changed lines of the file:
@@
 REF
 Wire Wire Line
-	12650 2850 12650 2750
-Wire Wire Line
-	12850 2450 12850 2350
+	12450 2850 12450 2750
 Wire Wire Line
 	12650 2450 12650 2350
+Wire Wire Line
+	12450 2450 12450 2350
 Connection ~ 12650 2350
-Wire Wire Line
-	12650 2350 12850 2350
 Wire Wire Line
 	11200 2250 10750 2250
@@
 L power:GND #PWR018
 U 1 1 60FB20EF
-P 12750 3250
-F 0 "#PWR018" H 12750 3000 50  0001 C CNN
-F 1 "GND" H 12750 3100 50  0000 C CNN
-F 2 "" H 12750 3250 50  0001 C CNN
-F 3 "" H 12750 3250 50  0001 C CNN
-	1    12750 3250
+P 12550 3250
+F 0 "#PWR018" H 12550 3000 50  0001 C CNN
+F 1 "GND" H 12550 3100 50  0000 C CNN
+F 2 "" H 12550 3250 50  0001 C CNN
+F 3 "" H 12550 3250 50  0001 C CNN
+	1    12550 3250
 	1    0    0    -1
 $EndComp
@@
 ATTEN-
 Wire Wire Line
-	12850 2750 12850 2850
+	12650 2750 12650 2850
 Connection ~ 8550 3250
 Connection ~ 8850 1450
@@
 P 2300 1600
 F 0 "C3" H 2450 1650 50  0000 L CNN
-F 1 "2.2uF 63V FILM" H 2450 1550 50  0000 L CNN
-F 2 "Capacitor_THT:C_Rect_L13.5mm_W5.0mm_P10.00mm_FKS3_FKP3_MKS4" H 2338 1450 50  0001 C CNN
+F 1 "1uF 100V FILM" H 2450 1550 50  0000 L CNN
+F 2 "Capacitor_THT:C_Rect_L7.2mm_W7.2mm_P5.00mm_FKS2_FKP2_MKS2_MKP2" H 2338 1450 50  0001 C CNN
 F 3 "~" H 2300 1600 50  0001 C CNN
-F 4 "R60DF4220506AJ" V 2300 1600 50  0001 C CNN "MPN"
+F 4 "R82EC4100SH70J" V 2300 1600 50  0001 C CNN "MPN"
 	1    2300 1600
 	-1   0    0    -1
@@
 $EndComp
 $Comp
-L Switch:SW_SPDT SW3
+L Switch:SW_DPDT_x2 SW3
 U 1 1 60F99B6D
-P 12750 3050
-F 0 "SW3" V 12750 3250 50  0000 L CNN
-F 1 "SPDT" V 12650 3250 50  0000 L CNN
-F 2 "high-gain-diff-probe:SW_TE_1825263-2_DPDT" H 12750 3050 50  0001 C CNN
-F 3 "http://switches-connectors-custom.cwind.com/Asset/GF-626-0061_2D%20DRAWING.PDF" H 12750 3050 50  0001 C CNN
-F 4 "Low Pass Enable" V 12850 3250 50  0000 L CNN "Name"
-F 5 "1825263-2" V 12750 3050 50  0001 C CNN "MPN"
-	1    12750 3050
+P 12550 3050
+F 0 "SW3" V 12550 3250 50  0000 L CNN
+F 1 "SPDT" V 12450 3250 50  0000 L CNN
+F 2 "high-gain-diff-probe:SW_TE_1825263-2_DPDT" H 12550 3050 50  0001 C CNN
+F 3 "http://switches-connectors-custom.cwind.com/Asset/GF-626-0061_2D%20DRAWING.PDF" H 12550 3050 50  0001 C CNN
+F 4 "Low Pass Enable" V 12650 3250 50  0000 L CNN "Name"
+F 5 "1825263-2" V 12550 3050 50  0001 C CNN "MPN"
+	1    12550 3050
 	0    -1   -1   0
 $EndComp
@@
 L Device:C C20
 U 1 1 6095342E
-P 12850 2600
-F 0 "C20" H 12965 2646 50  0000 L CNN
-F 1 "8.2nF" H 12965 2555 50  0000 L CNN
-F 2 "Capacitor_SMD:C_0603_1608Metric_Pad1.05x0.95mm_HandSolder" H 12888 2450 50  0001 C CNN
-F 3 "~" H 12850 2600 50  0001 C CNN
-F 4 "GRM1885C1H822JA01D" H 12850 2600 50  0001 C CNN "MPN"
-	1    12850 2600
+P 12650 2600
+F 0 "C20" V 12700 2650 50  0000 L CNN
+F 1 "8.2nF" V 12700 2350 50  0000 L CNN
+F 2 "Capacitor_SMD:C_0603_1608Metric_Pad1.05x0.95mm_HandSolder" H 12688 2450 50  0001 C CNN
+F 3 "~" H 12650 2600 50  0001 C CNN
+F 4 "GRM1885C1H822JA01D" H 12650 2600 50  0001 C CNN "MPN"
+	1    12650 2600
 	1    0    0    -1
 $EndComp
@@
 L Device:C C18
 U 1 1 60952944
-P 12650 2600
-F 0 "C18" H 12765 2646 50  0000 L CNN
-F 1 "20pF DNP" H 12765 2555 50  0000 L CNN
-F 2 "Capacitor_SMD:C_0603_1608Metric_Pad1.05x0.95mm_HandSolder" H 12688 2450 50  0001 C CNN
-F 3 "~" H 12650 2600 50  0001 C CNN
-	1    12650 2600
+P 12450 2600
+F 0 "C18" H 12565 2646 50  0000 L CNN
+F 1 "20pF DNP" H 12565 2555 50  0000 L CNN
+F 2 "Capacitor_SMD:C_0603_1608Metric_Pad1.05x0.95mm_HandSolder" H 12488 2450 50  0001 C CNN
+F 3 "~" H 12450 2600 50  0001 C CNN
+	1    12450 2600
 	-1   0    0    -1
 $EndComp
@@
 P 2300 4150
 F 0 "C4" H 2450 4200 50  0000 L CNN
-F 1 "2.2uF 63V FILM" H 2450 4100 50  0000 L CNN
-F 2 "Capacitor_THT:C_Rect_L13.5mm_W5.0mm_P10.00mm_FKS3_FKP3_MKS4" H 2338 4000 50  0001 C CNN
+F 1 "1uF 100V FILM" H 2450 4100 50  0000 L CNN
+F 2 "Capacitor_THT:C_Rect_L7.2mm_W7.2mm_P5.00mm_FKS2_FKP2_MKS2_MKP2" H 2338 4000 50  0001 C CNN
 F 3 "~" H 2300 4150 50  0001 C CNN
-F 4 "R60DF4220506AJ" V 2300 4150 50  0001 C CNN "MPN"
+F 4 "R82EC4100SH70J" V 2300 4150 50  0001 C CNN "MPN"
 	1    2300 4150
 	-1   0    0    1
@@
 	11700 4650 12200 4650
 Wire Wire Line
-	12400 2350 12650 2350
+	12400 2350 12450 2350
 Wire Wire Line
 	12100 2350 12000 2350
@@
 	1    0    0    -1
 $EndComp
-Wire Wire Line
-	13300 2350 12850 2350
-Connection ~ 12850 2350
 Wire Wire Line
 	13900 2450 14000 2450
@@
 F 3 "~" H 14250 5250 50  0001 C CNN
 F 4 "Fine Offset" V 13950 5250 50  0000 C CNN "Name"
-F 5 "PTV09A-4015U-B503" H 14250 5250 50  0001 C CNN "MPN"
+F 5 "PTV09A-4025F-B503" H 14250 5250 50  0001 C CNN "MPN"
 	1    14250 5250
 	0    1    -1   0
@@
 F 3 "~" H 14250 3900 50  0001 C CNN
 F 4 "Coarse Offset" V 13950 3900 50  0000 C CNN "Name"
-F 5 "PTV09A-4015U-B503" H 14250 3900 50  0001 C CNN "MPN"
+F 5 "PTV09A-4025F-B503" H 14250 3900 50  0001 C CNN "MPN"
 	1    14250 3900
 	0    1    1    0
@@
 Wire Wire Line
 	4600 900  4800 900
-Text Notes 12050 3600 0    50   ~ 0
+Text Notes 11900 3800 0    50   ~ 0
 TODO: Connect frame of switches to GND
+Connection ~ 12450 2350
+Wire Wire Line
+	12450 2350 12650 2350
+Wire Wire Line
+	12650 2350 13300 2350
 $EndSCHEMATC

Commit message: Tweaks
Other:
- moved on the sheet: C18, C20, SW3A
Changed lines of the file:
@@
 REF
 Wire Wire Line
-	12450 2850 12450 2750
+	12650 2850 12650 2750
+Wire Wire Line
+	12850 2450 12850 2350
 Wire Wire Line
 	12650 2450 12650 2350
-Wire Wire Line
-	12450 2450 12450 2350
 Connection ~ 12650 2350
 Wire Wire Line
@@
 L power:GND #PWR018
 U 1 1 60FB20EF
-P 12550 3250
-F 0 "#PWR018" H 12550 3000 50  0001 C CNN
-F 1 "GND" H 12550 3100 50  0000 C CNN
-F 2 "" H 12550 3250 50  0001 C CNN
-F 3 "" H 12550 3250 50  0001 C CNN
-	1    12550 3250
+P 12750 3250
+F 0 "#PWR018" H 12750 3000 50  0001 C CNN
+F 1 "GND" H 12750 3100 50  0000 C CNN
+F 2 "" H 12750 3250 50  0001 C CNN
+F 3 "" H 12750 3250 50  0001 C CNN
+	1    12750 3250
 	1    0    0    -1
 $EndComp
@@
 ATTEN-
 Wire Wire Line
-	12650 2750 12650 2850
+	12850 2750 12850 2850
 Connection ~ 8550 3250
 Connection ~ 8850 1450
@@
 L Switch:SW_DPDT_x2 SW3
 U 1 1 60F99B6D
-P 12550 3050
-F 0 "SW3" V 12550 3250 50  0000 L CNN
-F 1 "SPDT" V 12450 3250 50  0000 L CNN
-F 2 "high-gain-diff-probe:SW_TE_1825263-2_DPDT" H 12550 3050 50  0001 C CNN
-F 3 "http://switches-connectors-custom.cwind.com/Asset/GF-626-0061_2D%20DRAWING.PDF" H 12550 3050 50  0001 C CNN
-F 4 "Low Pass Enable" V 12650 3250 50  0000 L CNN "Name"
-F 5 "1825263-2" V 12550 3050 50  0001 C CNN "MPN"
-	1    12550 3050
+P 12750 3050
+F 0 "SW3" V 12750 3250 50  0000 L CNN
+F 1 "SPDT" V 12650 3250 50  0000 L CNN
+F 2 "high-gain-diff-probe:SW_TE_1825263-2_DPDT" H 12750 3050 50  0001 C CNN
+F 3 "http://switches-connectors-custom.cwind.com/Asset/GF-626-0061_2D%20DRAWING.PDF" H 12750 3050 50  0001 C CNN
+F 4 "Low Pass Enable" V 12850 3250 50  0000 L CNN "Name"
+F 5 "1825263-2" V 12750 3050 50  0001 C CNN "MPN"
+	1    12750 3050
 	0    -1   -1   0
 $EndComp
@@
 L Device:C C20
 U 1 1 6095342E
+P 12850 2600
+F 0 "C20" V 12900 2650 50  0000 L CNN
+F 1 "8.2nF" V 12900 2350 50  0000 L CNN
+F 2 "Capacitor_SMD:C_0603_1608Metric_Pad1.05x0.95mm_HandSolder" H 12888 2450 50  0001 C CNN
+F 3 "~" H 12850 2600 50  0001 C CNN
+F 4 "GRM1885C1H822JA01D" H 12850 2600 50  0001 C CNN "MPN"
+	1    12850 2600
+	1    0    0    -1
+$EndComp
+$Comp
+L Device:C C18
+U 1 1 60952944
 P 12650 2600
-F 0 "C20" V 12700 2650 50  0000 L CNN
-F 1 "8.2nF" V 12700 2350 50  0000 L CNN
+F 0 "C18" H 12765 2646 50  0000 L CNN
+F 1 "20pF DNP" H 12765 2555 50  0000 L CNN
 F 2 "Capacitor_SMD:C_0603_1608Metric_Pad1.05x0.95mm_HandSolder" H 12688 2450 50  0001 C CNN
 F 3 "~" H 12650 2600 50  0001 C CNN
-F 4 "GRM1885C1H822JA01D" H 12650 2600 50  0001 C CNN "MPN"
 	1    12650 2600
-	1    0    0    -1
-$EndComp
-$Comp
-L Device:C C18
-U 1 1 60952944
-P 12450 2600
-F 0 "C18" H 12565 2646 50  0000 L CNN
-F 1 "20pF DNP" H 12565 2555 50  0000 L CNN
-F 2 "Capacitor_SMD:C_0603_1608Metric_Pad1.05x0.95mm_HandSolder" H 12488 2450 50  0001 C CNN
-F 3 "~" H 12450 2600 50  0001 C CNN
-	1    12450 2600
 	-1   0    0    -1
 $EndComp
@@
 	11700 4650 12200 4650
 Wire Wire Line
-	12400 2350 12450 2350
-Wire Wire Line
 	12100 2350 12000 2350
 $Comp
@@
 Text Notes 11900 3800 0    50   ~ 0
 TODO: Connect frame of switches to GND
-Connection ~ 12450 2350
-Wire Wire Line
-	12450 2350 12650 2350
-Wire Wire Line
-	12650 2350 13300 2350
+Wire Wire Line
+	12650 2350 12850 2350
+Connection ~ 12850 2350
+Wire Wire Line
+	12850 2350 13300 2350
+Wire Wire Line
+	12400 2350 12650 2350
 $EndSCHEMATC
