File: high-gain-diff-probe.kicad_pcb (KiCad board)
At the start: 2 copper layers, 106 parts, among them J1 BANANA, J2 BNC, J3 BANANA, J4 BNC, J5 BNC, J6 POWER, Q1 BCV49, Q2 BCV48, SW1 MB04L1NCGD, SW2 MB04L1NCGD, SW3 GF-626-0061, SW4 GF-626-0061, U1 AD8428BRZ, U2 ADA4004, U3 BUF634A, U4 LM393, U5 LM393, U6 LM393

Commit message: Begin layout
Parts:
- D13, D14, D4, D5, D7, D8: value 1N4001 -> S1A; footprint Diode_THT:D_DO-41_SOD81_P10.16mm_Horizontal -> Diode_SMD:D_SMA_Handsoldering
- D15, D16, D17, D6: footprint LED_SMD:LED_0603_1608Metric_Pad1.05x0.95mm_HandSolder -> LED_THT:LED_D3.0mm
- J1, J3: footprint Connector:Banana_Jack_1Pin -> Connector:CalTest_CT3151
- RV2: footprint Potentiometer_THT:Potentiometer_Bourns_3296Y_Vertical -> Potentiometer_THT:Potentiometer_Piher_PT-6-V_Vertical
- moved D4 195.5 mm to (217.0, 110.0)
- moved D5 184.0 mm to (206.0, 110.0), turned to 180 degrees
- moved D8 182.2 mm to (217.0, 116.0), turned to 180 degrees
- moved J6 178.3 mm to (227.0, 110.0)
- moved J5 174.5 mm to (222.0, 133.0), turned to 270 degrees
- moved SW3 171.2 mm to (192.0, 145.0)
- moved D7 161.6 mm to (206.0, 116.0)
- moved SW4 157.4 mm to (183.0, 81.0)
- moved U3 150.6 mm to (207.0, 133.0)
- moved BT1 149.4 mm to (214.0, 104.0), turned to 90 degrees
- moved R16 145.5 mm to (215.0, 133.0), turned to 180 degrees
- moved BT4 143.6 mm to (214.0, 76.0), turned to 90 degrees
- moved BT2 140.4 mm to (214.0, 94.6), turned to 90 degrees
- moved SW2 136.8 mm to (172.0, 155.0)
- moved D11 134.5 mm to (150.0, 40.0), turned to 180 degrees
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Connections:
- net Net-(J5-Pad1) renamed /OUT

Commit message: Continue layout
Parts:
- J1, J3: footprint Connector:CalTest_CT3151 -> high-gain-diff-probe:CalTest_CT3151_Vertical
- moved J2 78.2 mm to (103.0, 88.0)
- moved R5 63.0 mm to (133.0, 98.5)
- moved R1 62.8 mm to (127.0, 98.5)
- moved C5 61.0 mm to (133.0, 96.5)
- moved C1 60.8 mm to (127.0, 96.5)
- moved R3 60.4 mm to (130.0, 78.0)
- moved C3 59.4 mm to (130.0, 88.0)
- moved J1 56.1 mm to (111.0, 89.0)
- moved C16 55.6 mm to (137.0, 148.0)
- moved C17 55.6 mm to (124.0, 151.0)
- moved C19 55.6 mm to (135.0, 139.0)
- moved R14 55.6 mm to (125.0, 138.0)
- moved R15 55.6 mm to (125.0, 142.0)
- moved RV2 55.6 mm to (128.0, 143.0)
- moved U2 55.6 mm to (130.0, 149.0)
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Routing:
- net /IN+: track 0.00 -> 56.4 mm
- net /HiZ+: track 0.00 -> 9.60 mm
- net Net-(C2-Pad1): track 0.00 -> 4.25 mm
- net Net-(R2-Pad1): track 0.00 -> 4.18 mm
Other:
- board outline added: 110 x 60 mm
- board text added: "Banana standard spacing is 0.75""

Commit message: Implement boost power
Parts:
- removed BT2, BT3, BT4: 9V, Connector_Wire:SolderWire-0.5sqmm_1x02_P4.6mm_D0.9mm_OD2.1mm_Relief
- removed D10, D9: 16V, Diode_SMD:D_SMF
- removed D13, D14, D8: S1A, Diode_SMD:D_SMA_Handsoldering
- removed J1, J3: BANANA, high-gain-diff-probe:CalTest_CT3151_Vertical
- removed Q1: BCV49, Package_TO_SOT_SMD:SOT-89-3_Handsoldering
- removed Q2: BCV48, Package_TO_SOT_SMD:SOT-89-3_Handsoldering
- removed SW1: MB04L1NCGD, high-gain-diff-probe:SW_DPNT_CK_M
- added C38: 1uF, Capacitor_SMD:C_0603_1608Metric_Pad1.05x0.95mm_HandSolder, F.Cu at (340.1, 72.6)
- added C39: 1uF, Capacitor_SMD:C_0603_1608Metric_Pad1.05x0.95mm_HandSolder, F.Cu at (350.5, 77.5)
- added C40: DNP, Capacitor_SMD:C_0603_1608Metric_Pad1.05x0.95mm_HandSolder, F.Cu at (367.1, 61.0)
- added C41: 1uF, Capacitor_SMD:C_0603_1608Metric_Pad1.05x0.95mm_HandSolder, F.Cu at (371.0, 36.0)
- added C42: 10pF, Capacitor_SMD:C_0603_1608Metric_Pad1.05x0.95mm_HandSolder, F.Cu at (380.9, 31.0)
- added C43: 1uF, Capacitor_SMD:C_0603_1608Metric_Pad1.05x0.95mm_HandSolder, F.Cu at (378.0, 35.0)
- added C44: 1uF, Capacitor_SMD:C_0603_1608Metric_Pad1.05x0.95mm_HandSolder, F.Cu at (376.0, 23.0)
- added C45: 10uF, Capacitor_SMD:C_0805_2012Metric_Pad1.15x1.40mm_HandSolder, F.Cu at (356.6, 52.5)
- added D18: S1A, Diode_SMD:D_SMA_Handsoldering, F.Cu at (121.0, 96.0)
- added D19: S1A, Diode_SMD:D_SMA_Handsoldering, F.Cu at (121.0, 105.0)
- added F1: 62mA 250V, Fuse:Fuseholder_Cylinder-5x20mm_Schurter_FAB_0031-355x_Horizontal_Closed, F.Cu at (116.5, 72.1)
- added F2: 62mA 250V, Fuse:Fuseholder_Cylinder-5x20mm_Schurter_FAB_0031-355x_Horizontal_Closed, F.Cu at (116.5, 128.5)
- added F3: 1A Fast, Fuse:Fuse_0805_2012Metric_Pad1.15x1.40mm_HandSolder, F.Cu at (351.6, 69.7)
- added F4: 1A Fast, Fuse:Fuse_0805_2012Metric_Pad1.15x1.40mm_HandSolder, F.Cu at (364.2, 55.8)
- added JP2: TERM, Connector_PinHeader_2.54mm:PinHeader_1x03_P2.54mm_Vertical, F.Cu at (351.9, 53.4)
- added JP3: TERM, Connector_PinHeader_2.54mm:PinHeader_1x03_P2.54mm_Vertical, F.Cu at (364.1, 46.9)
- added K1: FTR-B3GA4.5Z, Relay_SMD:Relay_Fujitsu_FTR-B3S, F.Cu at (113.0, 96.0)
- added K2: FTR-B3GA4.5Z, Relay_SMD:Relay_Fujitsu_FTR-B3S, F.Cu at (113.0, 105.0)
- added L1: 22uH, Inductor_SMD:L_Taiyo-Yuden_NR-40xx_HandSoldering, F.Cu at (368.0, 28.0)
- added L2: 22uH, Inductor_SMD:L_Taiyo-Yuden_NR-40xx_HandSoldering, F.Cu at (368.0, 33.0)
- added R28: 1M, Resistor_SMD:R_0603_1608Metric_Pad0.98x0.95mm_HandSolder, F.Cu at (376.0, 26.0)
- added R29: 83k, Resistor_SMD:R_0603_1608Metric_Pad0.98x0.95mm_HandSolder, F.Cu at (381.0, 27.0)
- added R30: 200, Resistor_SMD:R_0603_1608Metric_Pad0.98x0.95mm_HandSolder, F.Cu at (360.6, 68.4)
- added R31: 50, Resistor_SMD:R_0603_1608Metric_Pad0.98x0.95mm_HandSolder, F.Cu at (340.1, 75.1)
- added R32: DNP, Resistor_SMD:R_0603_1608Metric_Pad0.98x0.95mm_HandSolder, F.Cu at (374.5, 50.4)
- added R33: 10k, Resistor_SMD:R_0603_1608Metric_Pad0.98x0.95mm_HandSolder, F.Cu at (355.8, 73.4)
- added R34: 845, Resistor_SMD:R_0603_1608Metric_Pad0.98x0.95mm_HandSolder, F.Cu at (342.1, 70.1)
- added RV3: 200, Potentiometer_THT:Potentiometer_Bourns_3296Y_Vertical, F.Cu at (358.7, 42.0)
- added RV4: 200, Potentiometer_THT:Potentiometer_Bourns_3296Y_Vertical, F.Cu at (342.6, 63.7)
- added SW6: SPDT, high-gain-diff-probe:SW_CW_GF-626_DPDT, F.Cu at (143.0, 141.0)
- added U10: LM66100, Package_TO_SOT_SMD:Texas_R-PDSO-G6, F.Cu at (373.0, 73.0)
- added U11: LDL212, Package_SO:SO-8_3.9x4.9mm_P1.27mm, F.Cu at (311.0, 47.0)
- added U12: MC79M15, Package_TO_SOT_SMD:TO-252-2, F.Cu at (367.0, 80.0)
- added U7: AD8671, Package_SO:SOIC-8_3.9x4.9mm_P1.27mm, F.Cu at (194.0, 134.0)
- added U8: LT3463, Package_DFN_QFN:DFN-10-1EP_3x3mm_P0.5mm_EP1.65x2.38mm_ThermalVias, F.Cu at (375.6, 30.4)
- added U9: LM66100, Package_TO_SOT_SMD:Texas_R-PDSO-G6, F.Cu at (373.0, 66.0)
- BT1: value 9V -> 3xAA; footprint Connector_Wire:SolderWire-0.5sqmm_1x02_P4.6mm_D0.9mm_OD2.1mm_Relief -> Battery:BatteryHolder_Keystone_2479_3xAAA; moved to B.Cu
- C1, C2: value 27pF -> 20pF
- C10, C9: value DNP -> 1nF
- C11, C12: value 10p -> DNP
- C13: value 120p -> DNP
- C14, C15, C16, C17, C19, C21, C22, C25, C26, C27, C30, C31, C32, C33, C34, C35, C36, C37: value 100nF -> 1uF
- C18: value 120pF -> 20pF DNP
- C20: value 33nF -> 8.2nF
- C28, C29: value 47uF -> 1uF; footprint Capacitor_THT:CP_Radial_D6.3mm_P2.50mm -> Capacitor_SMD:C_0603_1608Metric_Pad1.05x0.95mm_HandSolder
- C3, C4: value 1uF FILM -> 2.2uF 63V FILM; footprint high-gain-diff-probe:C_6054_WIMA -> Capacitor_THT:C_Rect_L13.5mm_W5.0mm_P10.00mm_FKS3_FKP3_MKS4
- C5, C6: value 27pF -> 8-30pF; footprint Capacitor_SMD:C_0603_1608Metric_Pad1.05x0.95mm_HandSolder -> Capacitor_SMD:C_Trimmer_Voltronics_JZ
- C7, C8: value 3-10pF -> 8-30pF
- D4: value S1A -> DSS13UTR; footprint Diode_SMD:D_SMA_Handsoldering -> Diode_SMD:D_SOD-123F
- D5, D7: value S1A -> US1A; footprint Diode_SMD:D_SMA_Handsoldering -> Diode_SMD:D_SMA
- J6: value POWER -> USB_B; footprint Connector_PinHeader_2.54mm:PinHeader_1x03_P2.54mm_Horizontal -> Connector_USB:USB_B_Lumberg_2411_02_Horizontal
- R1, R6: value 475k -> 990k 0.1%; footprint Resistor_SMD:R_0603_1608Metric_Pad0.98x0.95mm_HandSolder -> Resistor_SMD:R_1206_3216Metric_Pad1.30x1.75mm_HandSolder
- R10: value 2k -> 1M 0.1%
- R11, R12: value 33 -> 33 0.1%
- R13, R3: value 50 -> 200
- R18: value 4.7k -> 15k
- R19: value 4.7k -> 75k
- R2: value 475k -> 200; footprint Resistor_SMD:R_0603_1608Metric_Pad0.98x0.95mm_HandSolder -> Resistor_SMD:R_1210_3225Metric_Pad1.30x2.65mm_HandSolder
- R20: value 100 -> 1M
- R21: value 100 -> 15k
- R22, R23, R27: value 25.6k -> 4.7k
- R25: value 25.6k -> 10k
- R4: value 50 -> 1M; footprint Resistor_SMD:R_1210_3225Metric_Pad1.30x2.65mm_HandSolder -> Resistor_SMD:R_0603_1608Metric_Pad0.98x0.95mm_HandSolder
- R5: value 475k -> 1M
- R7, R8: value 49.9k -> 10k 0.1%
- R9: value 154 -> 1M 0.1%
- RV1: value 500 -> 200; footprint Potentiometer_THT:Potentiometer_Bourns_3266W_Vertical -> Potentiometer_THT:Potentiometer_Bourns_3296Y_Vertical
- SW2: value MB04L1NCGD -> MB05L1NCGD
- SW3: value GF-626-0061 -> SPDT
- SW4: value GF-626-0061 -> MFS201N-4-Z; footprint high-gain-diff-probe:SW_CW_GF-626_DPDT -> high-gain-diff-probe:SW_Nidec_DPDT_MFS201N−4-Z
- U2: value ADA4004 -> OP1177AR
- moved R4 240.6 mm to (362.8, 61.1), turned to 0 degrees
- moved R5 225.6 mm to (356.2, 65.8), turned to 0 degrees
- moved R20 206.7 mm to (381.0, 33.0), turned to 0 degrees
- moved C28 196.7 mm to (374.5, 52.9)
- moved C29 195.1 mm to (379.8, 48.4)
- moved R18 192.5 mm to (364.0, 58.5), turned to 0 degrees
- moved D12 191.4 mm to (358.0, 98.0), turned to 0 degrees
- moved R10 190.4 mm to (335.7, 74.9), turned to 0 degrees
- moved R19 189.8 mm to (381.0, 29.0), turned to 0 degrees
- moved C30 185.4 mm to (349.8, 87.0)
- moved C31 185.4 mm to (357.8, 87.0)
- moved C23 184.5 mm to (348.8, 92.7)
- moved C24 184.5 mm to (356.8, 92.7)
- moved D11 177.6 mm to (350.0, 98.0), turned to 0 degrees
- moved R9 175.4 mm to (335.7, 72.3), turned to 0 degrees
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Connections:
- BT1 pad 1: Net-(BT1-Pad1) -> /AAA
- BT1 pad 2: Net-(BT1-Pad2) -> GND
- C1 pad 2: /IN- -> Net-(C1-Pad2)
- C10 pad 2: ATTEN+ -> Net-(C10-Pad2)
- C2 pad 2: /IN+ -> Net-(C2-Pad2)
- C25 pad 1: Net-(C25-Pad1) -> /+16V6
- C26 pad 2: Net-(C26-Pad2) -> /-16V6
- C29 pad 1: GND -> Net-(C29-Pad1)
- C29 pad 2: Net-(C29-Pad2) -> GND
- C3 pad 1: /AC- -> Net-(C3-Pad1)
- C3 pad 2: /IN- -> Net-(C3-Pad2)
- C4 pad 1: /AC+ -> Net-(C4-Pad1)
- C4 pad 2: /IN+ -> Net-(C4-Pad2)
- C5 pad 1: /HiZ- -> Net-(C5-Pad1)
- C6 pad 1: /HiZ+ -> Net-(C10-Pad2)
- C7 pad 1: ATTEN- -> Net-(C5-Pad1)
- C8 pad 2: ATTEN+ -> Net-(C10-Pad2)
- C9 pad 1: ATTEN- -> Net-(C5-Pad1)
- D4 pad 1: Net-(D4-Pad1) -> Net-(C41-Pad1)
- D4 pad 2: Net-(D4-Pad2) -> /-16V6
- D5 pad 1: Net-(D4-Pad1) -> /+16V6
- D5 pad 2: Net-(BT1-Pad1) -> +15V
- D6 pad 2: Net-(C25-Pad1) -> +15V
- D7 pad 1: Net-(BT4-Pad2) -> -15V
- D7 pad 2: Net-(D7-Pad2) -> /-16V6
- J6 pad 1: Net-(D4-Pad2) -> Net-(F4-Pad2)
- J6 pad 2: GND -> (no net)
- J6 pad 3: Net-(D8-Pad1) -> (no net)
- R1 pad 1: Net-(R1-Pad1) -> Net-(C5-Pad1)
- R1 pad 2: /IN- -> Net-(C1-Pad2)
- R10 pad 1: /RG_500X -> Net-(JP3-Pad2)
- R10 pad 2: Net-(R10-Pad2) -> GND
- R17 pad 2: GND -> -15V
- R18 pad 1: Net-(C25-Pad1) -> Net-(R18-Pad1)
- R18 pad 2: Net-(C28-Pad1) -> Net-(R18-Pad2)
- R19 pad 1: Net-(C29-Pad2) -> Net-(R19-Pad1)
- R19 pad 2: Net-(C26-Pad2) -> Net-(C42-Pad1)
- R2 pad 1: Net-(R2-Pad1) -> Net-(F1-Pad2)
- R2 pad 2: /IN+ -> /IN-
- R20 pad 1: Net-(Q1-Pad1) -> Net-(C42-Pad1)
- R20 pad 2: Net-(C28-Pad1) -> /-16V6
- R21 pad 1: Net-(C29-Pad2) -> Net-(R21-Pad1)
- R3 pad 1: /LoZ- -> Net-(F2-Pad2)
- R3 pad 2: /IN- -> /IN+
- R4 pad 1: /LoZ+ -> Net-(C3-Pad1)
- R4 pad 2: /IN+ -> Net-(K1-Pad3)
- R5 pad 1: /HiZ- -> Net-(C4-Pad1)
- R5 pad 2: Net-(R1-Pad1) -> Net-(K2-Pad3)
- R6 pad 1: /HiZ+ -> Net-(C10-Pad2)
- R6 pad 2: Net-(R2-Pad1) -> Net-(C2-Pad2)
- R7 pad 1: ATTEN- -> Net-(C5-Pad1)
- R8 pad 2: ATTEN+ -> Net-(C10-Pad2)
- R9 pad 1: /RG_50X -> Net-(JP2-Pad2)
- R9 pad 2: Net-(R9-Pad2) -> GND
- SW2 pad 10: (no net) -> ATTEN_EN
- SW2 pad 2: /RG_500X -> /RG_100X
- SW2 pad 3: /RG_50X -> /RG_10X
- SW2 pad 4: (no net) -> /RG_100X
- SW2 pad 5: (no net) -> /RG_10X
- SW2 pad 7: Net-(R10-Pad2) -> (no net)
- SW2 pad 8: Net-(R9-Pad2) -> (no net)
- SW2 pad 9: (no net) -> ATTEN_EN
- SW2 pad B: /FIL+ -> +5V
- SW4 pad 1: (no net) -> Net-(R18-Pad1)
- SW4 pad 2: Net-(D4-Pad1) -> Net-(C29-Pad1)
- SW4 pad 3: Net-(C25-Pad1) -> (no net)
- SW4 pad 4: (no net) -> Net-(R21-Pad1)
- SW4 pad 5: Net-(D7-Pad2) -> Net-(C28-Pad1)
- SW4 pad 6: Net-(C26-Pad2) -> (no net)
- U1 pad 6: /REF -> Net-(SW6-Pad2)
- U3 pad 3: SE_SIG -> Net-(C40-Pad2)
Routing:
- net /IN+: track 56.4 -> 0.00 mm
- net /HiZ+: track 9.60 -> 0.00 mm
- net Net-(C2-Pad1): track 4.25 -> 0.00 mm
- net Net-(R2-Pad1): track 4.18 -> 0.00 mm
Other:
- board text removed: "Banana standard spacing is 0.75""

Commit message: Simplify power
Parts:
- removed BT1: 3xAA, Battery:BatteryHolder_Keystone_2479_3xAAA
- removed C17, C22, C25, C26, C28, C29, C39, C41, C43, C44: 1uF, Capacitor_SMD:C_0603_1608Metric_Pad1.05x0.95mm_HandSolder
- removed C23, C24: 47uF, Capacitor_THT:CP_Radial_D6.3mm_P2.50mm
- removed C42: 10pF, Capacitor_SMD:C_0603_1608Metric_Pad1.05x0.95mm_HandSolder
- removed C45: 10uF, Capacitor_SMD:C_0805_2012Metric_Pad1.15x1.40mm_HandSolder
- removed D4: DSS13UTR, Diode_SMD:D_SOD-123F
- removed D5: US1A, Diode_SMD:D_SMA
- removed F3: 1A Fast, Fuse:Fuse_0805_2012Metric_Pad1.15x1.40mm_HandSolder
- removed J6: USB_B, Connector_USB:USB_B_Lumberg_2411_02_Horizontal
- removed JP2, JP3: TERM, Connector_PinHeader_2.54mm:PinHeader_1x03_P2.54mm_Vertical
- removed L1, L2: 22uH, Inductor_SMD:L_Taiyo-Yuden_NR-40xx_HandSoldering
- removed R28: 1M, Resistor_SMD:R_0603_1608Metric_Pad0.98x0.95mm_HandSolder
- removed R29: 83k, Resistor_SMD:R_0603_1608Metric_Pad0.98x0.95mm_HandSolder
- removed R33: 10k, Resistor_SMD:R_0603_1608Metric_Pad0.98x0.95mm_HandSolder
- removed R34: 845, Resistor_SMD:R_0603_1608Metric_Pad0.98x0.95mm_HandSolder
- removed U10, U9: LM66100, Package_TO_SOT_SMD:Texas_R-PDSO-G6
- removed U11: LDL212, Package_SO:SO-8_3.9x4.9mm_P1.27mm
- removed U12: MC79M15, Package_TO_SOT_SMD:TO-252-2
- added GD1: DNP, high-gain-diff-probe:GDT_Bourns_2031, F.Cu at (124.0, 74.0)
- added GD2: DNP, high-gain-diff-probe:GDT_Bourns_2031, F.Cu at (124.0, 131.0)
- added J1: 30V DC IN, Connector_BarrelJack:BarrelJack_CUI_PJ-063AH_Horizontal, F.Cu at (240.0, 33.2)
- added Q1: 2N3906, Package_TO_SOT_THT:TO-92_Inline, F.Cu at (266.4, 34.5)
- added RV5: 50k, Potentiometer_THT:Potentiometer_Bourns_PTV09A-1_Single_Vertical, F.Cu at (253.8, 68.8)
- added SW1: MB04L1NCGD, high-gain-diff-probe:SW_DPNT_CK_M, F.Cu at (228.6, 66.9)
- C15: value 1uF -> 47uF; footprint Capacitor_SMD:C_0603_1608Metric_Pad1.05x0.95mm_HandSolder -> Capacitor_THT:CP_Radial_D8.0mm_P5.00mm
- K1, K2: value FTR-B3GA4.5Z -> FTR-B3SA012Z
- R14: value 10k -> 1k
- R15: value 10k -> 100k
- R19: value 75k -> 15k
- R20: value 1M -> 1k; footprint Resistor_SMD:R_0603_1608Metric_Pad0.98x0.95mm_HandSolder -> Capacitor_SMD:C_0603_1608Metric_Pad1.05x0.95mm_HandSolder
- R21: value 15k -> 250k; footprint Resistor_SMD:R_0603_1608Metric_Pad0.98x0.95mm_HandSolder -> Capacitor_SMD:C_0603_1608Metric_Pad1.05x0.95mm_HandSolder
- RV2: footprint Potentiometer_THT:Potentiometer_Piher_PT-6-V_Vertical -> Potentiometer_THT:Potentiometer_Bourns_PTV09A-1_Single_Vertical
- SW3, SW6: footprint high-gain-diff-probe:SW_CW_GF-626_DPDT -> Button_Switch_THT:SW_E-Switch_EG2219_DPDT_Angled
- SW4: value MFS201N-4-Z -> MB04L1NCGD; footprint high-gain-diff-probe:SW_Nidec_DPDT_MFS201N−4-Z -> high-gain-diff-probe:SW_DPNT_CK_M
- U8: value LT3463 -> BUF634A; footprint Package_DFN_QFN:DFN-10-1EP_3x3mm_P0.5mm_EP1.65x2.38mm_ThermalVias -> Package_SO:SOIC-8-1EP_3.9x4.9mm_P1.27mm_EP2.41x3.81mm_ThermalVias
- moved R20 163.7 mm to (223.0, 76.0)
- moved U8 139.2 mm to (237.7, 49.5)
- moved R21 129.1 mm to (227.3, 76.0)
- moved R19 124.9 mm to (256.8, 42.0)
- moved R18 120.4 mm to (244.1, 47.5)
- moved C15 95.0 mm to (249.0, 36.0), turned to 0 degrees
- moved SW4 95.0 mm to (244.3, 66.9)
- moved C30 81.3 mm to (273.8, 116.0)
- moved C31 81.3 mm to (281.8, 116.0)
- moved C38 81.3 mm to (264.1, 101.6)
- moved C40 81.3 mm to (291.1, 90.0)
- moved D11 81.3 mm to (274.0, 127.0)
- moved D12 81.3 mm to (282.0, 127.0)
- moved D7 81.3 mm to (290.0, 115.0)
- moved F4 81.3 mm to (288.2, 84.8)
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Connections:
- C14 pad 2: GND -> -15V
- C15 pad 1: GND -> +15V
- C16 pad 2: GND -> -15V
- C21 pad 2: GND -> -15V
- C30 pad 2: GND -> Net-(C30-Pad2)
- C31 pad 1: GND -> Net-(C30-Pad2)
- C38 pad 2: GND -> -15V
- D11 pad 2: GND -> Net-(C30-Pad2)
- D12 pad 1: GND -> Net-(C30-Pad2)
- D18 pad 2: GND -> Net-(D18-Pad2)
- D19 pad 1: ATTEN_EN -> Net-(D18-Pad2)
- D19 pad 2: GND -> -15V
- D7 pad 1: -15V -> Net-(D7-Pad1)
- D7 pad 2: /-16V6 -> Net-(D7-Pad2)
- F4 pad 1: Net-(C29-Pad1) -> +15V
- F4 pad 2: Net-(F4-Pad2) -> Net-(D7-Pad1)
- K1 pad 8: GND -> Net-(D18-Pad2)
- K2 pad 1: ATTEN_EN -> Net-(D18-Pad2)
- K2 pad 8: GND -> -15V
- R10 pad 1: Net-(JP3-Pad2) -> Net-(R10-Pad1)
- R14 pad 1: +15V -> Net-(C19-Pad2)
- R15 pad 2: -15V -> Net-(C19-Pad2)
- R17 pad 2: -15V -> Net-(C30-Pad2)
- R18 pad 1: Net-(R18-Pad1) -> +15V
- R19 pad 1: Net-(R19-Pad1) -> Net-(R18-Pad2)
- R19 pad 2: Net-(C42-Pad1) -> -15V
- R20 pad 1: Net-(C42-Pad1) -> ATTEN_EN
- R20 pad 2: /-16V6 -> Net-(Q1-Pad3)
- RV2 pad 1: Net-(R15-Pad1) -> -15V
- RV2 pad 2: Net-(C19-Pad2) -> Net-(R14-Pad2)
- RV2 pad 3: Net-(R14-Pad2) -> +15V
- SW2 pad 10: ATTEN_EN -> Net-(R21-Pad1)
- SW2 pad 9: ATTEN_EN -> Net-(R21-Pad1)
- SW2 pad B: +5V -> -15V
- SW4 pad 1: Net-(R18-Pad1) -> Net-(C4-Pad1)
- SW4 pad 2: Net-(C29-Pad1) -> GND
- SW4 pad 3: (no net) -> Net-(R10-Pad1)
- SW4 pad 4: Net-(R21-Pad1) -> (no net)
- SW4 pad 5: Net-(C28-Pad1) -> (no net)
- SW4 pad 6: (no net) -> Net-(SW4-Pad6)
- U8 pad 1: /+16V6 -> (no net)
- U8 pad 2: Net-(L1-Pad2) -> (no net)
- U8 pad 3: +5V -> Net-(R18-Pad2)
- U8 pad 4: Net-(C41-Pad2) -> -15V
- U8 pad 5: Net-(C41-Pad1) -> (no net)
- U8 pad 6: Net-(C42-Pad1) -> Net-(C30-Pad2)
- U8 pad 7: Net-(R19-Pad1) -> +15V
- U8 pad 8: +5V -> (no net)
- U8 pad 9: +5V -> (no net)

Commit message: Layout
Parts:
- removed C32, C33, C35, C36: 1uF, Capacitor_SMD:C_0603_1608Metric_Pad1.05x0.95mm_HandSolder
- removed D15, D16: LED, LED_THT:LED_D3.0mm
- removed R22, R23: 4.7k, Resistor_SMD:R_0603_1608Metric_Pad0.98x0.95mm_HandSolder
- removed U4, U5: LM393, Package_SO:SOIC-8_3.9x4.9mm_P1.27mm
- C14, D18, D19: moved to B.Cu
- C37: value 1uF -> 100nF
- F1, F2: footprint Fuse:Fuseholder_Cylinder-5x20mm_Schurter_FAB_0031-355x_Horizontal_Closed -> high-gain-diff-probe:Fuseholder_Schurter_0031.8273
- moved R4 175.3 mm to (111.5, 89.0), turned to 270 degrees
- moved R5 158.4 mm to (123.0, 114.0), turned to 90 degrees
- moved RV3 154.5 mm to (140.5, 131.3), turned to 90 degrees
- moved Q1 152.8 mm to (142.5, 124.0), turned to 90 degrees
- moved R30 143.4 mm to (146.5, 136.0), turned to 90 degrees
- moved R9 139.7 mm to (122.0, 78.0), turned to 180 degrees
- moved R10 134.8 mm to (125.0, 108.0), turned to 180 degrees
- moved R32 131.1 mm to (176.0, 126.0), turned to 180 degrees
- moved SW4 122.3 mm to (132.0, 115.5)
- moved C34 115.2 mm to (212.8, 99.7)
- moved C37 115.2 mm to (205.8, 87.7)
- moved D17 115.2 mm to (208.8, 88.7)
- moved R24 115.2 mm to (204.8, 98.7)
- moved R25 115.2 mm to (204.8, 94.8)
- moved R26 115.2 mm to (204.8, 90.7)
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Connections:
- U6 pad 2: SE_SIG -> Net-(R24-Pad1)
- U6 pad 3: Net-(R24-Pad1) -> SE_SIG
- U6 pad 5: SE_SIG -> Net-(R25-Pad1)
- U6 pad 6: Net-(R25-Pad1) -> SE_SIG
Routing:
- net Net-(K2-Pad2): track 0.00 -> 6.14 mm
- net Net-(K1-Pad2): track 0.00 -> 6.14 mm
Other:
- board size 110 x 60 mm -> 110 x 80 mm

Commit message: More layout
Parts:
- removed D6: LED, LED_THT:LED_D3.0mm
- removed R17: 15k, Resistor_SMD:R_0603_1608Metric_Pad0.98x0.95mm_HandSolder
- added C17: 1uF, Capacitor_SMD:C_0603_1608Metric_Pad1.05x0.95mm_HandSolder, B.Cu at (158.8, 96.2)
- added C22: 1uF, Capacitor_SMD:C_0603_1608Metric_Pad1.05x0.95mm_HandSolder, B.Cu at (158.8, 103.8)
- added C23: 1uF, Capacitor_SMD:C_0603_1608Metric_Pad1.05x0.95mm_HandSolder, F.Cu at (183.4, 77.9)
- added R22: 10k 0.1%, Resistor_SMD:R_0603_1608Metric_Pad0.98x0.95mm_HandSolder, F.Cu at (144.0, 80.4)
- added R23: 10k 0.1%, Resistor_SMD:R_0603_1608Metric_Pad0.98x0.95mm_HandSolder, F.Cu at (154.6, 76.0)
- added RV6: 200, Potentiometer_THT:Potentiometer_Bourns_3296Y_Vertical, F.Cu at (152.8, 79.4)
- C1, C2: value 20pF -> 22pF; footprint Capacitor_SMD:C_0603_1608Metric_Pad1.05x0.95mm_HandSolder -> Capacitor_SMD:C_0805_2012Metric_Pad1.15x1.40mm_HandSolder
- C15: footprint Capacitor_THT:CP_Radial_D8.0mm_P5.00mm -> Capacitor_SMD:CP_Elec_6.3x7.7
- C16, C34, C38: moved to B.Cu
- Q1: value 2N3906 -> MMBT3906; footprint Package_TO_SOT_THT:TO-92_Inline -> Package_TO_SOT_SMD:SOT-23
- SW3, SW6: footprint Button_Switch_THT:SW_E-Switch_EG2219_DPDT_Angled -> high-gain-diff-probe:SW_TE_1825263-2_DPDT
- moved D7 54.2 mm to (187.2, 63.0)
- moved C15 49.9 mm to (179.9, 66.3), turned to 180 degrees
- moved J1 48.7 mm to (187.4, 71.2)
- moved R19 45.1 mm to (178.4, 70.9), turned to 180 degrees
- moved F4 44.6 mm to (192.0, 63.0)
- moved R18 41.7 mm to (182.0, 70.9), turned to 180 degrees
- moved SW6 40.5 mm to (157.6, 87.6), turned to 180 degrees
- moved U8 38.9 mm to (179.8, 75.9), turned to 270 degrees
- moved C31 37.7 mm to (176.1, 77.9)
- moved C27 35.9 mm to (178.2, 84.8), turned to 180 degrees
- moved D12 35.2 mm to (175.5, 82.6), turned to 180 degrees
- moved C30 33.6 mm to (180.2, 80.6), turned to 180 degrees
- moved U6 30.9 mm to (182.2, 98.6), turned to 270 degrees
- moved C34 30.6 mm to (182.2, 98.6)
- moved R26 29.2 mm to (177.6, 101.2), turned to 0 degrees
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Connections:
- C18 pad 1: SE_SIG -> Net-(C18-Pad1)
- C20 pad 1: SE_SIG -> Net-(C18-Pad1)
- C30 pad 2: Net-(C30-Pad2) -> GND
- C31 pad 1: Net-(C30-Pad2) -> GND
- C8 pad 1: GND -> Net-(C10-Pad2)
- C8 pad 2: Net-(C10-Pad2) -> GND
- D11 pad 2: Net-(C30-Pad2) -> GND
- D12 pad 1: Net-(C30-Pad2) -> GND
- D7 pad 1: Net-(D7-Pad1) -> +15V
- F4 pad 1: +15V -> Net-(D7-Pad2)
- F4 pad 2: Net-(D7-Pad1) -> Net-(F4-Pad2)
- J1 pad 1: Net-(D7-Pad2) -> Net-(F4-Pad2)
- J1 pad MP: (no net) -> Net-(J1-PadMP)
- JP1 pad 1: Net-(JP1-Pad1) -> (no net)
- K1 pad 3: Net-(K1-Pad3) -> ATTEN-
- K1 pad 6: ATTEN- -> Net-(K1-Pad6)
- Q1 pad 1: +15V -> Net-(Q1-Pad1)
- Q1 pad 2: Net-(Q1-Pad2) -> +15V
- R13 pad 1: SE_SIG -> Net-(C18-Pad1)
- R14 pad 1: Net-(C19-Pad2) -> Net-(R14-Pad1)
- R15 pad 2: Net-(C19-Pad2) -> Net-(R14-Pad1)
- R21 pad 2: Net-(Q1-Pad2) -> Net-(Q1-Pad1)
- R4 pad 2: Net-(K1-Pad3) -> Net-(K1-Pad6)
- RV1 pad 1: Net-(R8-Pad1) -> Net-(R7-Pad2)
- RV1 pad 3: Net-(R7-Pad2) -> Net-(R8-Pad1)
- SW1 pad 1: Net-(C3-Pad1) -> Net-(SW1-Pad1)
- SW1 pad 2: GND -> Net-(SW1-Pad1)
- SW1 pad 3: Net-(R9-Pad1) -> Net-(C3-Pad2)
- SW1 pad 4: (no net) -> Net-(C3-Pad2)
- SW1 pad 6: Net-(SW1-Pad6) -> Net-(C3-Pad1)
- SW1 pad 7: Net-(SW1-Pad6) -> GND
- SW1 pad 8: Net-(C3-Pad2) -> Net-(R9-Pad1)
- SW1 pad 9: Net-(C3-Pad2) -> (no net)
- SW1 pad A: Net-(SW1-Pad6) -> Net-(K1-Pad6)
- SW1 pad B: Net-(K1-Pad3) -> Net-(SW1-Pad1)
- SW6 pad 1: GND -> Net-(R14-Pad1)
- SW6 pad 2: Net-(SW6-Pad2) -> Net-(C19-Pad2)
- SW6 pad 3: /REF -> Net-(RV6-Pad2)
- U1 pad 6: Net-(SW6-Pad2) -> /REF
- U3 pad 1: Net-(JP1-Pad1) -> (no net)
- U3 pad 9: (no net) -> -15V
- U6 pad 3: SE_SIG -> /OUT
- U6 pad 6: SE_SIG -> /OUT
- U7 pad 3: SE_SIG -> Net-(C18-Pad1)
- U8 pad 6: Net-(C30-Pad2) -> GND
- U8 pad 9: (no net) -> -15V
Routing:
- net Net-(D18-Pad2): track 0.00 -> 25.5 mm, vias 0 -> 2
- net -15V: track 0.00 -> 24.7 mm, vias 0 -> 7
- net Net-(F2-Pad2): track 0.00 -> 20.6 mm
- net +15V: track 0.00 -> 20.6 mm, vias 0 -> 6
- net Net-(F1-Pad2): track 0.00 -> 20.3 mm
- net GND: track 0.00 -> 19.8 mm, vias 0 -> 10
- net Net-(R14-Pad1): track 0.00 -> 18.2 mm
- net Net-(C4-Pad2): track 0.00 -> 17.5 mm
- net Net-(C5-Pad1): track 0.00 -> 17.3 mm
- net Net-(C3-Pad2): track 0.00 -> 17.0 mm
- net Net-(C10-Pad2): track 0.00 -> 16.6 mm
- net Net-(F4-Pad2): track 0.00 -> 9.08 mm
- net Net-(SW4-Pad6): track 0.00 -> 8.47 mm
- net Net-(SW1-Pad1): track 0.00 -> 8.47 mm
- net ATTEN+: track 0.00 -> 7.56 mm
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- added copper zone on In2.Cu, net +15V
- added copper zone on B.Cu, net -15V
- added copper zone on In1.Cu, net GND
Other:
- copper layers 2 -> 4

Commit message: More layout
Parts:
- added C24: 47uF, Capacitor_SMD:CP_Elec_6.3x7.7, F.Cu at (190.1, 82.9)
- added C25: 47uF, Capacitor_SMD:CP_Elec_6.3x7.7, F.Cu at (171.6, 82.5)
- added C26: 1uF, Capacitor_SMD:C_0603_1608Metric_Pad1.05x0.95mm_HandSolder, F.Cu at (165.8, 92.2)
- added C28: 1uF, Capacitor_SMD:C_0603_1608Metric_Pad1.05x0.95mm_HandSolder, F.Cu at (163.3, 82.7)
- added C29: 1uF, Capacitor_SMD:C_0603_1608Metric_Pad1.05x0.95mm_HandSolder, F.Cu at (185.7, 100.6)
- added C32: 1uF, Capacitor_SMD:C_0603_1608Metric_Pad1.05x0.95mm_HandSolder, F.Cu at (174.7, 103.2)
- added C33: 1uF, Capacitor_SMD:C_0603_1608Metric_Pad1.05x0.95mm_HandSolder, F.Cu at (183.6, 80.6)
- added C35: 1uF, Capacitor_SMD:C_0603_1608Metric_Pad1.05x0.95mm_HandSolder, F.Cu at (176.1, 73.8)
- added JP2: BANDWIDTH, Jumper:SolderJumper-2_P1.3mm_Open_TrianglePad1.0x1.5mm, F.Cu at (184.2, 73.5)
- moved SW3 40.1 mm to (171.3, 91.0)
- moved D17 37.9 mm to (192.0, 126.0), turned to 90 degrees
- moved C37 37.2 mm to (176.0, 122.0), turned to 270 degrees
- moved R27 34.9 mm to (196.5, 123.0)
- moved C20 28.9 mm to (175.3, 96.9), turned to 90 degrees
- moved R24 28.7 mm to (183.5, 124.1), turned to 270 degrees
- moved R25 22.5 mm to (183.5, 120.5), turned to 270 degrees
- moved C34 21.4 mm to (179.8, 119.9), turned to 0 degrees
- moved U6 21.4 mm to (179.8, 119.9), turned to 90 degrees
- moved R32 21.1 mm to (174.7, 100.5)
- moved C40 20.7 mm to (180.2, 97.3)
- moved U7 20.7 mm to (180.2, 101.3)
- moved C38 20.7 mm to (180.2, 101.9)
- moved R9 17.6 mm to (128.9, 91.3), turned to 0 degrees
- moved D12 17.5 mm to (191.8, 89.1)
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Connections:
- J1 pad MP: Net-(J1-PadMP) -> GND
- JP1 pad 1: (no net) -> Net-(JP1-Pad1)
- U3 pad 1: (no net) -> Net-(JP1-Pad1)
- U8 pad 1: (no net) -> Net-(JP2-Pad1)
Routing:
- net /FIL+: track 0.00 -> 34.0 mm, vias 0 -> 1
- net ATTEN-: track 4.59 -> 36.6 mm, vias 0 -> 2
- net ATTEN+: track 7.56 -> 38.7 mm, vias 0 -> 2
- net /RG_10X: track 0.00 -> 24.8 mm
- net Net-(C3-Pad1): track 4.24 -> 23.5 mm, vias 0 -> 2
- net /FIL-: track 0.00 -> 18.7 mm
- net Net-(C3-Pad2): track 17.0 -> 33.6 mm
- net Net-(K2-Pad3): track 3.06 -> 19.4 mm
- net Net-(K1-Pad6): track 3.06 -> 18.6 mm
- net Net-(C4-Pad2): track 17.5 -> 31.7 mm
- net /RG_100X: track 0.00 -> 14.1 mm
- net Net-(R21-Pad1): track 0.00 -> 9.48 mm
- net Net-(C4-Pad1): track 4.24 -> 13.4 mm
- net Net-(R30-Pad2): track 0.00 -> 8.69 mm
- net -15V: track 24.7 -> 31.5 mm
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