File: high-gain-diff-probe.kicad_pcb (KiCad board)
At the start: 4 copper layers, 110 x 80 mm, 107 parts, among them J1 30V DC IN, J2 BNC, J4 BNC, J5 BNC, K1 FTR-B3SA012Z, K2 FTR-B3SA012Z, Q1 MMBT3906, SW1 MB04L1NCGD, SW2 MB05L1NCGD, SW3 SPDT, SW4 MB04L1NCGD, SW6 SPDT, U1 AD8428BRZ, U2 OP1177AR, U3 BUF634A, U6 LM393, U7 AD8671, U8 BUF634A

Commit message: Tweaks
Parts:
- removed D18, D19: S1A, Diode_SMD:D_SMA_Handsoldering
- removed D7: US1A, Diode_SMD:D_SMA
- added D4: DSS15, Diode_SMD:D_SOD-123F, F.Cu at (186.5, 63.0)
- added D5: DSS15, Diode_SMD:D_SOD-123F, B.Cu at (106.5, 94.5)
- added D6: DSS15, Diode_SMD:D_SOD-123F, B.Cu at (106.5, 105.5)
- Q1: moved to B.Cu
- R20: value 1k -> 1k 1/4W; footprint Capacitor_SMD:C_0603_1608Metric_Pad1.05x0.95mm_HandSolder -> Resistor_SMD:R_1206_3216Metric_Pad1.30x1.75mm_HandSolder; moved to B.Cu
- R21: value 250k -> 100k; footprint Capacitor_SMD:C_0603_1608Metric_Pad1.05x0.95mm_HandSolder -> Resistor_SMD:R_0603_1608Metric_Pad0.98x0.95mm_HandSolder
- moved Q1 55.3 mm to (102.5, 101.0)
- moved R20 54.8 mm to (106.5, 99.5)
- moved F4 1.00 mm to (191.0, 63.0), turned to 0 degrees
Connections:
- SW2 pad 6: (no net) -> GND
- SW2 pad 7: (no net) -> GND
- SW2 pad 8: (no net) -> GND
- SW2 pad B: -15V -> GND
Routing:
- net -15V: track 31.5 -> 23.8 mm
- net GND: track 23.4 -> 30.2 mm
- net Net-(R21-Pad1): track 9.48 -> 3.34 mm
- net Net-(D5-Pad2): track 25.5 -> 23.2 mm
- net Net-(Q1-Pad1): track 1.90 -> 0.00 mm
- net Net-(D4-Pad2): track 3.22 -> 2.07 mm
- net Net-(F4-Pad2): track 9.08 -> 10.1 mm
- net Net-(Q1-Pad3): track 2.03 -> 3.02 mm
- net ATTEN_EN: track 5.47 -> 6.42 mm
